Commit message: Update robot.urdf

File: src/robot/models/robot.urdf (robot description, URDF)
Before this commit: robot robot, 5 links, 4 joints
Links:
- removed link BL_Wheel
- removed link BR_Wheel
- removed link FL_Wheel
- removed link FR_Wheel
- removed link Frame
- added link base_footprint
- added link base_link; collision box size=${base_length} ${base_width} ${base_height}; visual mesh filename=package://robot/meshes/FrameDetailed.stl
- added link gps_link
- added link imu_link
Joints:
- removed joint BL_Axel
- removed joint BR_Axel
- removed joint FL_Axel
- removed joint FR_Axel
- added joint base_joint: type fixed, parent base_footprint, child base_link, origin xyz=0.0 0.0 ${(wheel_radius+wheel_zoff)} rpy=0 0 0
- added joint gps_joint: type fixed, parent base_link, child gps_link, origin xyz=0.10 0 0.05 rpy=0 0 0
- added joint imu_joint: type fixed, parent base_link, child imu_link, origin xyz=-0.10 0 0.05 rpy=0 0 0
